File: schematics/dmx-shutter.sch (KiCad schematic (older format))
At the start: 12 parts

Commit message: KiCad version update things
Parts:
- C? (x3): symbol C -> dmx-shutter-rescue:C
- D?: symbol LED -> dmx-shutter-rescue:LED
- IC?: symbol ATMEGA88PA-P -> dmx-shutter-rescue:ATMEGA88PA-P
- K?: symbol XLR3 -> dmx-shutter-rescue:XLR3
- P?: symbol CONN_01X02 -> dmx-shutter-rescue:CONN_01X02
- Q?: symbol BC547 -> dmx-shutter-rescue:BC547
- R? (x2): symbol R -> dmx-shutter-rescue:R
- U?: symbol SN75176B -> dmx-shutter-rescue:SN75176B
- Y?: symbol Crystal -> dmx-shutter-rescue:Crystal
Changed lines of the file:
@@
-EESchema Schematic File Version 2
-LIBS:power
-LIBS:device
-LIBS:transistors
-LIBS:conn
-LIBS:linear
-LIBS:regul
-LIBS:74xx
-LIBS:cmos4000
-LIBS:adc-dac
-LIBS:memory
-LIBS:xilinx
-LIBS:microcontrollers
-LIBS:dsp
-LIBS:microchip
-LIBS:analog_switches
-LIBS:motorola
-LIBS:texas
-LIBS:intel
-LIBS:audio
-LIBS:interface
-LIBS:digital-audio
-LIBS:philips
-LIBS:display
-LIBS:cypress
-LIBS:siliconi
-LIBS:opto
-LIBS:atmel
-LIBS:contrib
-LIBS:valves
-LIBS:oturpe-kicad-lib
-EELAYER 25 0
+EESchema Schematic File Version 4
+LIBS:dmx-shutter-cache
+EELAYER 30 0
 EELAYER END
 $Descr A4 11693 8268
@@
 $EndDescr
 $Comp
-L ATMEGA88PA-P IC?
+L dmx-shutter-rescue:ATMEGA88PA-P IC?
 U 1 1 573C797E
 P 3000 3500
@@
 $EndComp
 $Comp
-L GND #PWR?
+L power:GND #PWR?
 U 1 1 573C7AE5
 P 2100 4700
@@
 	2100 4700 2100 4600
 $Comp
-L +5V #PWR?
+L power:+5V #PWR?
 U 1 1 573C7BB7
 P 2100 2400
@@
 	2100 2700 2100 2400
 $Comp
-L C C?
+L dmx-shutter-rescue:C C?
 U 1 1 573C7BD4
 P 1950 2550
@@
 $EndComp
 $Comp
-L GND #PWR?
+L power:GND #PWR?
 U 1 1 573C7C11
 P 1950 2700
@@
 	2100 2400 1950 2400
 $Comp
-L +5V #PWR?
+L power:+5V #PWR?
 U 1 1 573C7DD3
 P 5350 3300
@@
 $EndComp
 $Comp
-L GND #PWR?
+L power:GND #PWR?
 U 1 1 573C7E04
 P 5250 3700
@@
 	5350 3700 5250 3700
 Wire Wire Line
-	5250 3700 5250 3400
+	5250 3700 5250 3600
 Wire Wire Line
 	5250 3400 5350 3400
 Connection ~ 5250 3600
 $Comp
-L SN75176B U?
+L dmx-shutter-rescue:SN75176B U?
 U 1 1 573C7A9C
 P 5800 3200
@@
 	4000 4000 5350 4000
 $Comp
-L XLR3 K?
+L dmx-shutter-rescue:XLR3 K?
 U 1 1 573C838A
 P 6600 2850
@@
 $EndComp
 $Comp
-L GND #PWR?
+L power:GND #PWR?
 U 1 1 573C8449
 P 6250 2850
@@
 	6950 2850 6950 3400
 $Comp
-L R R?
+L dmx-shutter-rescue:R R?
 U 1 1 573C874B
 P 3850 2100
@@
 $EndComp
 $Comp
-L LED D?
+L dmx-shutter-rescue:LED D?
 U 1 1 573C88B9
 P 3500 2100
@@
 	4000 2400 4000 2100
 $Comp
-L GND #PWR?
+L power:GND #PWR?
 U 1 1 573C88F7
 P 3300 2100
@@
 $EndComp
 $Comp
-L BC547 Q?
+L dmx-shutter-rescue:BC547 Q?
 U 1 1 573C8C23
 P 6500 4700
@@
 $EndComp
 $Comp
-L CONN_01X02 P?
+L dmx-shutter-rescue:CONN_01X02 P?
 U 1 1 573C8E60
 P 6800 4250
@@
 TODO: How should this external \ndvd player tray button be connected?
 $Comp
-L GND #PWR?
+L power:GND #PWR?
 U 1 1 573C8ECE
 P 6600 4900
@@
 $EndComp
 $Comp
-L R R?
+L dmx-shutter-rescue:R R?
 U 1 1 573C8FB5
 P 6150 4700
@@
 $EndComp
 $Comp
-L Crystal Y?
+L dmx-shutter-rescue:Crystal Y?
 U 1 1 573C903F
 P 4350 3050
@@
 	4850 4700 6000 4700
 $Comp
-L C C?
+L dmx-shutter-rescue:C C?
 U 1 1 573C9911
 P 4800 2900
@@
 $EndComp
 $Comp
-L C C?
+L dmx-shutter-rescue:C C?
 U 1 1 573C9AEE
 P 4800 3200
@@
 $EndComp
 $Comp
-L GND #PWR?
+L power:GND #PWR?
 U 1 1 573C9B35
 P 4600 3050
@@
 Wire Wire Line
 	4100 2900 4350 2900
+Wire Wire Line
+	5250 3600 5250 3400
 $EndSCHEMATC
